Commit message: initial fork commit

File: franka_description/robots/common/franka_robot.xacro (robot description, xacro)
@@ -69,4 +69,16 @@
         </plugin>
         <self_collide>true</self_collide>
+        <!-- ADDED GRIPPER -->
+        <gripper name="test_gripper">
+          <palm_link>${arm_id}_hand</palm_link>
+          <gripper_link>${arm_id}_leftfinger</gripper_link>
+          <gripper_link>${arm_id}_rightfinger</gripper_link>
+          <grasp_check>
+            <detach_steps>10</detach_steps>
+            <attach_steps>10</attach_steps>
+            <min_cintact_count>4</min_cintact_count>
+          </grasp_check>
+        </gripper>
+        <!-- END ADDED GRIPPER -->
       </gazebo>
     </xacro:if>

File: franka_description/robots/panda/panda.urdf.xacro (robot description, xacro)
@@ -32,5 +32,5 @@
   <link name="camera_mount_rotation"></link>
   <joint name="camera_mount_base_joint" type="fixed">
-   <parent link="panda_hand_tcp"/>
+   <parent link="panda_hand_sc"/>
    <child link="camera_mount_base"/>
    <origin rpy="0 0 0"/>
